File: RTCMemoryVoltageSourceAndBattery/RTCMemoryVoltageSourceAndBattery.kicad_pcb (KiCad board)
At the start: 2 copper layers, 16 parts, among them IC1 LM2597M-3.3_NOPB, IC2 MAX6326UR31+T, J1 Screw_Terminal_01x02, J2 Conn_01x02, J3 Conn_01x02, Q1 BD140, Q2 BS250

Commit message: Routed and labeled. Ready for Fab
Parts:
- IC2: moved to F.Cu
- J1: value Screw_Terminal_01x02 -> Conn_01x02; footprint TerminalBlock_Phoenix:TerminalBlock_Phoenix_MKDS-1,5-2-5.08_1x02_P5.08mm_Horizontal -> Connector_PinSocket_2.54mm:PinSocket_1x02_P2.54mm_Vertical
- moved J3 45.4 mm to (141.7, 81.9), turned to 180 degrees
- moved C4 38.1 mm to (106.5, 88.1)
- moved J2 31.1 mm to (141.7, 89.9), turned to 180 degrees
- moved J1 30.2 mm to (141.7, 97.8), turned to 180 degrees
- moved Q1 30.0 mm to (137.9, 97.8), turned to 90 degrees
- moved Q2 26.7 mm to (136.1, 83.8), turned to 90 degrees
- moved D2 25.9 mm to (123.0, 96.7), turned to 180 degrees
- moved C1 22.5 mm to (113.2, 84.6), turned to -90 degrees
- moved C2 18.4 mm to (125.2, 85.0), turned to -90 degrees
- moved R2 18.2 mm to (105.3, 84.4)
- moved IC2 17.4 mm to (136.8, 87.6)
- moved R1 16.9 mm to (134.1, 92.6), turned to -90 degrees
- moved D1 15.9 mm to (129.2, 79.4)
- moved IC1 15.4 mm to (119.2, 85.3)
- moved C3 15.3 mm to (119.6, 90.9)
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Routing:
- net GND: track 0.00 -> 220.9 mm, vias 0 -> 4
- net +3.3VP: track 0.00 -> 62.2 mm
- net Net-(D2-Pad1): track 0.00 -> 34.8 mm
- net +VDC: track 0.00 -> 31.5 mm
- net Net-(J2-Pad1): track 0.00 -> 9.34 mm
- net Net-(D1-Pad1): track 0.00 -> 9.23 mm
- net Net-(IC1-Pad1): track 0.00 -> 9.13 mm
- net Net-(IC2-Pad2): track 0.00 -> 5.49 mm
- net Net-(C2-Pad1): track 0.00 -> 4.17 mm
- net Net-(Q1-Pad3): track 0.00 -> 3.94 mm
- net Net-(Q1-Pad1): track 0.00 -> 3.78 mm
- net Net-(C1-Pad1): track 0.00 -> 3.30 mm
- added copper zone on B.Cu, net GND
Other:
- board outline added: 50.8 x 25.4 mm
- board text added: "GND"
- board text added: "VBat"
- board text added: "VDC"
- board text added: "VOut"
- board text added: "https://github.com/TJLTM/RTCMemoryVS"
