File: RTCMemoryVoltageSourceAndBattery/RTCMemoryVoltageSourceAndBattery.kicad_sch (KiCad schematic)
At the start: 12 parts, among them IC1 LM2597M-3.3_NOPB, J1 Screw_Terminal_01x02, Q1 IRF9Z34NPBF, U1 BK_HTC-15M

Commit message: continuing schem wip
Parts:
- removed Q1: IRF9Z34NPBF, SamacSys_Parts:TO254P469X1042X1967-3P, symbol SamacSys_Parts:IRF9Z34NPBF
- removed U1: BK_HTC-15M, SamacSys_Parts:BK_HTC-15M, symbol SamacSys_Parts:BK_HTC-15M
- added D2: 1N4001, Diode_THT:D_DO-41_SOD81_P10.16mm_Horizontal, symbol Diode:1N4001
- added IC2: MAX6326UR31+T, SOT95P237X112-3N, symbol Samac_Sys:MAX6326UR31+T
- added J2, J3: Conn_01x02, Connector_PinSocket_2.54mm:PinSocket_1x02_P2.54mm_Vertical, symbol Connector_Generic:Conn_01x02
- added Q1: BD140, Package_TO_SOT_THT:TO-126-3_Vertical, symbol Transistor_BJT:BD140
- added Q2: BS250, Package_TO_SOT_THT:TO-92_Inline, symbol Transistor_FET:BS250
Connections:
- net +3.3VP: now also D2.2 (A), IC2.3 (VCC)
- net +VDC: now also Q1.2 (C)
- net GND: now also IC2.1 (GND), J2.2 (Pin_2), J3.2 (Pin_2)
- net at R1.1: now also Q1.3 (B)
- net at J1.1 (Pin_1): now also Q1.1 (E)
- new net: D2.1 (K), J3.1 (Pin_1), Q2.3 (S)
- new net: J2.1 (Pin_1), Q2.1 (D)
- new net: IC2.2 (~{RESET}), Q2.2 (G)
Other:
- moved on the sheet: C1, C2, C3, C4, D1, IC1, J1, L1, R1, R2

Commit message: Routed and labeled. Ready for Fab
Parts:
- removed J1: Screw_Terminal_01x02, TerminalBlock_Phoenix:TerminalBlock_Phoenix_MKDS-1,5-2-5.08_1x02_P5.08mm_Horizontal, symbol Connector:Screw_Terminal_01x02
- added J1: Conn_01x02, Connector_PinSocket_2.54mm:PinSocket_1x02_P2.54mm_Vertical, symbol Connector_Generic:Conn_01x02
Connections:
- net GND: now also J1.2 (Pin_2)
- net at Q1.1 (E): now also J1.1 (Pin_1)
Changed lines of the file:
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@@
   )
   (symbol (lib_id "Connector_Generic:Conn_01x02") (at 98.425 115.57 0) (mirror y) (unit 1)
-    (in_bom yes) (on_board yes) (fields_autoplaced)
+    (in_bom yes) (on_board yes)
     (property "Reference" "J2" (id 0) (at 98.425 110.3335 0))
     (property "Value" "Conn_01x02" (id 1) (at 98.425 113.1086 0))
-    (property "Footprint" "Connector_PinSocket_2.54mm:PinSocket_1x02_P2.54mm_Vertical" (id 2) (at 98.425 115.57 0))
+    (property "Footprint" "Connector_PinSocket_2.54mm:PinSocket_1x02_P2.54mm_Vertical" (id 2) (at 99.06 132.08 0))
     (property "Datasheet" "~" (id 3) (at 98.425 115.57 0)
       (effects (font (size 1.27 1.27)) hide)
@@
     (pin "2")
     (pin "3")
-  )
-  (symbol (lib_id "Connector:Screw_Terminal_01x02") (at 23.495 38.735 0) (mirror y) (unit 1)
-    (in_bom yes) (on_board yes)
-    (property "Reference" "J1" (id 0) (at 25.5778 33.2232 0))
-    (property "Value" "Screw_Terminal_01x02" (id 1) (at 25.5778 35.5346 0))
-    (property "Footprint" "TerminalBlock_Phoenix:TerminalBlock_Phoenix_MKDS-1,5-2-5.08_1x02_P5.08mm_Horizontal" (id 2) (at 23.495 38.735 0)
-      (effects (font (size 1.27 1.27)) hide)
-    )
-    (property "Datasheet" "~" (id 3) (at 23.495 38.735 0)
-      (effects (font (size 1.27 1.27)) hide)
-    )
-    (pin "1")
-    (pin "2")
   )
   (symbol (lib_id "Device:R") (at 74.93 27.305 0) (unit 1)
@@
     (pin "8")
   )
+  (symbol (lib_id "Connector_Generic:Conn_01x02") (at 23.495 38.735 0) (mirror y) (unit 1)
+    (in_bom yes) (on_board yes) (fields_autoplaced)
+    (property "Reference" "J1" (id 0) (at 23.495 33.4985 0))
+    (property "Value" "Conn_01x02" (id 1) (at 23.495 36.2736 0))
+    (property "Footprint" "Connector_PinSocket_2.54mm:PinSocket_1x02_P2.54mm_Vertical" (id 2) (at 23.495 38.735 0))
+    (property "Datasheet" "~" (id 3) (at 23.495 38.735 0)
+      (effects (font (size 1.27 1.27)) hide)
+    )
+    (pin "1")
+    (pin "2")
+  )
   (symbol (lib_id "Transistor_FET:BS250") (at 112.395 113.03 90) (mirror x) (unit 1)
     (in_bom yes) (on_board yes) (fields_autoplaced)
@@
       (reference "IC2") (unit 1) (value "MAX6326UR31+T") (footprint "SOT95P237X112-3N")
     )
-    (path "/bbeb5660-87a7-4a13-be2a-0981978dab67"
-      (reference "J1") (unit 1) (value "Screw_Terminal_01x02") (footprint "TerminalBlock_Phoenix:TerminalBlock_Phoenix_MKDS-1,5-2-5.08_1x02_P5.08mm_Horizontal")
+    (path "/f48726b8-0a84-4a45-918f-9908a36bbb39"
+      (reference "J1") (unit 1) (value "Conn_01x02") (footprint "Connector_PinSocket_2.54mm:PinSocket_1x02_P2.54mm_Vertical")
     )
     (path "/a5936896-849b-42a6-ad04-ca5f7f31c73c"
